Commit message: Update

File: src/sweepi_description/urdf/camera.xacro (robot description, xacro)
@@ -37,36 +37,15 @@
     <origin xyz="${body_radius + camera_length / 2.0} 0 0" rpy="0 0 0"/>
   </joint>
-  <link name="camera_link_optical"/>
-  <joint name="camera_optical_joint" type="fixed">
+  <link name="camera_rgb_frame"/>
+  <joint name="camera_rgb_joint" type="fixed">
     <parent link="camera_link"/>
-    <child  link="camera_link_optical"/>
-    <origin xyz="0 0 0" rpy="${-pi/2} 0 ${-pi/2}"/>
+    <child  link="camera_rgb_frame"/>
+    <origin xyz="0 0 0" rpy="0 0 0"/>
   </joint>
-  <gazebo reference="camera_link">
-    <sensor name="camera" type="camera">
-      <camera>
-        <horizontal_fov>1.3962634</horizontal_fov>
-        <image>
-          <width>640</width>
-          <height>480</height>
-          <format>R8G8B8</format>
-        </image>
-        <clip>
-          <near>0.1</near>
-          <far>15</far>
-        </clip>
-        <noise>
-          <type>gaussian</type>
-          <mean>0.0</mean>
-          <stddev>0.007</stddev>
-        </noise>
-        <optical_frame_id>camera_link_optical</optical_frame_id>
-        <camera_info_topic>camera/camera_info</camera_info_topic>
-      </camera>
-      <always_on>1</always_on>
-      <update_rate>20</update_rate>
-      <visualize>true</visualize>
-      <topic>camera/image_raw</topic>
-    </sensor>
-  </gazebo>
+  <link name="camera_rgb_optical_frame"/>
+  <joint name="camera_rgb_optical_joint" type="fixed">
+    <parent link="camera_rgb_frame"/>
+    <child  link="camera_rgb_optical_frame"/>
+    <origin xyz="0 0 0" rpy="-1.57 0 -1.57"/>
+  </joint>
 </robot>

File: src/sweepi_description/urdf/lidar.xacro (robot description, xacro)
@@ -37,37 +37,3 @@
     <origin xyz="${lidar_offset_x} 0 ${body_height / 2.0 + lidar_height / 2.0}" rpy="0 0 0"/>
   </joint>
-  <gazebo reference="lidar_link">
-    <sensor name="rplidar_c1" type="gpu_lidar">
-      <topic>scan</topic>
-      <update_rate>10</update_rate>
-      <always_on>1</always_on>
-      <visualize>true</visualize>
-      <lidar>
-        <scan>
-          <horizontal>
-            <samples>720</samples>
-            <resolution>1</resolution>
-            <min_angle>-3.14159</min_angle>
-            <max_angle>3.14159</max_angle>
-          </horizontal>
-        </scan>
-        <range>
-          <min>0.05</min>
-          <max>12.0</max>
-          <resolution>0.005</resolution>
-        </range>
-        <noise>
-          <type>gaussian</type>
-          <mean>0.0</mean>
-          <stddev>0.001</stddev>
-        </noise>
-      </lidar>
-    </sensor>
-  </gazebo>
-  <gazebo>
-    <plugin name="gz::sim::systems::Sensors"
-            filename="gz-sim-sensors-system">
-      <render_engine>ogre2</render_engine>
-    </plugin>
-  </gazebo>
 </robot>

File: src/sweepi_description/urdf/robot_base.xacro (robot description, xacro)
@@ -65,7 +65,7 @@
       <collision>
         <geometry>
-          <sphere radius="${drive_wheel_radius}"/>
+          <cylinder radius="${drive_wheel_radius}" length="${drive_wheel_width}"/>
         </geometry>
-        <origin xyz="0 0 0" rpy="0 0 0"/>
+        <origin xyz="0 0 0" rpy="${pi / 2.0} 0 0"/>
       </collision>
       <xacro:cylinder_inertia
@@ -77,6 +77,6 @@
     </link>
   </xacro:macro>
+  <xacro:drive_wheel_link prefix="left"/>
   <xacro:drive_wheel_link prefix="right"/>
-  <xacro:drive_wheel_link prefix="left"/>
   <xacro:macro name="caster_link" params="prefix">
     <link name="${prefix}_caster_link">
@@ -130,16 +130,18 @@
     <origin xyz="0 0 ${base_joint_z}" rpy="0 0 0"/>
   </joint>
+  <!-- LEFT WHEEL JOINT - Axis should be Y (perpendicular to wheel width) -->
+  <joint name="base_left_wheel_joint" type="continuous">
+    <parent link="base_link"/>
+    <child  link="left_wheel_link"/>
+    <origin xyz="0 ${wheel_span / 2.0} ${wheel_z_offset}" rpy="0 0 0"/>
+    <axis xyz="0 1 0"/>
+    <dynamics damping="0.01" friction="0.01"/>
+  </joint>
+  <!-- RIGHT WHEEL JOINT - Axis should be Y (perpendicular to wheel width) -->
   <joint name="base_right_wheel_joint" type="continuous">
     <parent link="base_link"/>
     <child  link="right_wheel_link"/>
     <origin xyz="0 ${-(wheel_span / 2.0)} ${wheel_z_offset}" rpy="0 0 0"/>
-    <axis   xyz="0 1 0"/>
-    <dynamics damping="0.01" friction="0.01"/>
-  </joint>
-  <joint name="base_left_wheel_joint" type="continuous">
-    <parent link="base_link"/>
-    <child  link="left_wheel_link"/>
-    <origin xyz="0 ${wheel_span / 2.0} ${wheel_z_offset}" rpy="0 0 0"/>
-    <axis   xyz="0 1 0"/>
+    <axis xyz="0 1 0"/>
     <dynamics damping="0.01" friction="0.01"/>
   </joint>

File: src/sweepi_description/urdf/robot_base_gazebo.xacro (robot description, xacro)
@@ -1,4 +1,5 @@
 <?xml version="1.0"?>
 <robot xmlns:xacro="http://www.ros.org/wiki/xacro">
+  <!-- Friction for caster wheels -->
   <gazebo reference="front_caster_link">
     <mu1>0.1</mu1>
@@ -9,22 +10,25 @@
     <mu2>0.1</mu2>
   </gazebo>
- <gazebo>
-    <plugin
-      filename="gz-sim-diff-drive-system"
-      name="gz::sim::systems::DiffDrive">
+  <!-- Differential Drive Controller -->
+  <gazebo>
+    <plugin filename="gz-sim-diff-drive-system"
+            name="gz::sim::systems::DiffDrive">
       <left_joint>base_left_wheel_joint</left_joint>
       <right_joint>base_right_wheel_joint</right_joint>
-      <wheel_separation>0.30</wheel_separation>   <!-- match your URDF -->
-      <wheel_radius>0.025</wheel_radius>          <!-- match your URDF -->
+      <wheel_separation>0.300</wheel_separation>
+      <wheel_radius>0.025</wheel_radius>
+      <odom_publish_frequency>50</odom_publish_frequency>
+      <topic>/model/sweepi/cmd_vel</topic>
+      <odom_topic>/odom</odom_topic>
+      <tf_topic>/model/sweepi/tf</tf_topic>
       <frame_id>odom</frame_id>
       <child_frame_id>base_footprint</child_frame_id>
-      <topic>cmd_vel</topic>
-      <odom_topic>odom</odom_topic>
+      <max_linear_acceleration>1.0</max_linear_acceleration>
     </plugin>
   </gazebo>
-   <gazebo>
-    <plugin
-      filename="gz-sim-joint-state-publisher-system"
-      name="gz::sim::systems::JointStatePublisher">
+  <!-- Joint State Publisher -->
+  <gazebo>
+    <plugin filename="gz-sim-joint-state-publisher-system"
+            name="gz::sim::systems::JointStatePublisher">
       <joint_name>base_left_wheel_joint</joint_name>
       <joint_name>base_right_wheel_joint</joint_name>

File: src/sweepi_description/urdf/sweepi.urdf.xacro (robot description, xacro)
@@ -1,7 +1,12 @@
 <?xml version="1.0"?>
 <robot name="sweepi" xmlns:xacro="http://www.ros.org/wiki/xacro">
+  <!-- Include robot base definition -->
   <xacro:include filename="robot_base.xacro"/>
+  <!-- Include sensors (camera and lidar) -->
   <xacro:include filename="camera.xacro"/>
   <xacro:include filename="lidar.xacro"/>
+  <!-- Include Gazebo sensor plugins -->
+  <xacro:include filename="sensor_gazebo.xacro"/>
+  <!-- Include Gazebo base plugins and controller -->
   <xacro:include filename="robot_base_gazebo.xacro"/>
 </robot>

Commit message: Fix camera plugin

File: src/sweepi_description/urdf/camera.xacro (robot description, xacro)
@@ -37,15 +37,36 @@
     <origin xyz="${body_radius + camera_length / 2.0} 0 0" rpy="0 0 0"/>
   </joint>
-  <link name="camera_rgb_frame"/>
-  <joint name="camera_rgb_joint" type="fixed">
+  <link name="camera_link_optical"/>
+  <joint name="camera_optical_joint" type="fixed">
     <parent link="camera_link"/>
-    <child  link="camera_rgb_frame"/>
-    <origin xyz="0 0 0" rpy="0 0 0"/>
+    <child  link="camera_link_optical"/>
+    <origin xyz="0 0 0" rpy="${-pi/2} 0 ${-pi/2}"/>
   </joint>
-  <link name="camera_rgb_optical_frame"/>
-  <joint name="camera_rgb_optical_joint" type="fixed">
-    <parent link="camera_rgb_frame"/>
-    <child  link="camera_rgb_optical_frame"/>
-    <origin xyz="0 0 0" rpy="-1.57 0 -1.57"/>
-  </joint>
+  <gazebo reference="camera_link">
+    <sensor name="camera" type="camera">
+      <camera>
+        <horizontal_fov>1.3962634</horizontal_fov>
+        <image>
+          <width>640</width>
+          <height>480</height>
+          <format>R8G8B8</format>
+        </image>
+        <clip>
+          <near>0.1</near>
+          <far>15.0</far>
+        </clip>
+        <noise>
+          <type>gaussian</type>
+          <mean>0.0</mean>
+          <stddev>0.007</stddev>
+        </noise>
+        <optical_frame_id>camera_link_optical</optical_frame_id>
+        <camera_info_topic>camera/camera_info</camera_info_topic>
+      </camera>
+      <always_on>1</always_on>
+      <update_rate>20</update_rate>
+      <visualize>true</visualize>
+      <topic>camera/image_raw</topic>
+    </sensor>
+  </gazebo>
 </robot>

File: src/sweepi_description/urdf/sensor_gazebo.xacro (robot description, xacro)
@@ -1,43 +1,37 @@
 <?xml version="1.0"?>
 <robot xmlns:xacro="http://www.ros.org/wiki/xacro">
-  <gazebo reference="camera_link">
-    <sensor name="camera" type="camera">
-      <pose>0 0 0 0 0 0</pose>
+    <gazebo reference="camera_link">
+        <sensor name="camera" type="camera">
+            <camera>
+                <horizontal_fov>1.3962634</horizontal_fov>
+                <image>
+                    <width>640</width>
+                    <height>480</height>
+                    <format>R8G8B8</format>
+                </image>
+                <clip>
+                    <near>0.1</near>
+                    <far>15</far>
+                </clip>
+                <noise>
+                    <type>gaussian</type>
+                    <mean>0.0</mean>
+                    <stddev>0.007</stddev>
+                </noise>
+                <optical_frame_id>camera_link_optical</optical_frame_id>
+                <camera_info_topic>camera/camera_info</camera_info_topic>
+            </camera>
+            <always_on>1</always_on>
+            <update_rate>20</update_rate>
+            <visualize>true</visualize>
+            <topic>camera/image_raw</topic>
+        </sensor>
+    </gazebo>
+  <gazebo reference="lidar_link">
+    <sensor name="lidar_sensor" type="lidar">
+      <topic>scan</topic>
+      <update_rate>10</update_rate>
       <visualize>true</visualize>
-      <update_rate>30</update_rate>
-      <camera name="camera">
-        <horizontal_fov>1.047</horizontal_fov>
-        <image>
-          <width>640</width>
-          <height>480</height>
-          <format>R8G8B8</format>
-        </image>
-        <clip>
-          <near>0.02</near>
-          <far>300</far>
-        </clip>
-        <noise>
-          <type>gaussian</type>
-          <mean>0.0</mean>
-          <stddev>0.007</stddev>
-        </noise>
-      </camera>
-      <always_on>1</always_on>
-      <topic>/camera/image_raw</topic>
-    </sensor>
-  </gazebo>
-  <gazebo reference="camera_rgb_optical_frame">
-    <sensor name="camera_info" type="camera">
-      <always_on>1</always_on>
-      <update_rate>30</update_rate>
-      <topic>/camera/camera_info</topic>
-    </sensor>
-  </gazebo>
- <gazebo reference="lidar_link">
-    <sensor name="gpu_lidar" type="gpu_lidar">
-      <pose>0 0 0 0 0 0</pose>
-      <visualize>true</visualize>
-      <update_rate>10</update_rate>
-      <ray>
+      <lidar>
         <scan>
           <horizontal>
@@ -64,7 +58,5 @@
           <stddev>0.001</stddev>
         </noise>
-      </ray>
-      <always_on>1</always_on>
-      <topic>/scan</topic>
+      </lidar>
     </sensor>
   </gazebo>

File: src/sweepi_description/urdf/sweepi.urdf.xacro (robot description, xacro)
@@ -5,7 +5,7 @@
   <!-- Include sensors (camera and lidar) -->
   <xacro:include filename="camera.xacro"/>
-  <xacro:include filename="lidar.xacro"/>
+  <!-- <xacro:include filename="lidar.xacro"/> -->
   <!-- Include Gazebo sensor plugins -->
-  <xacro:include filename="sensor_gazebo.xacro"/>
+  <!-- <xacro:include filename="sensor_gazebo.xacro"/> -->
   <!-- Include Gazebo base plugins and controller -->
   <xacro:include filename="robot_base_gazebo.xacro"/>
