Commit message: update

File: src/sweepi_description/urdf/lidar.xacro (robot description, xacro)
@@ -32,4 +32,5 @@
       o_xyz="0 0 0" o_rpy="0 0 0"/>
   </link>
+  <link name="lidar_link_optical"/>
   <joint name="base_lidar_joint" type="fixed">
     <parent link="base_link"/>
@@ -37,39 +38,43 @@
     <origin xyz="${lidar_offset_x} 0 ${body_height / 2.0 + lidar_height / 2.0}" rpy="0 0 0"/>
   </joint>
-  <!-- <gazebo>
-    <plugin
-      filename="gz-sim-sensors-system"
-      name="gz::sim::systems::Sensors">
-      <render_engine>ogre2</render_engine>
-    </plugin>
-  </gazebo> -->
+  <joint name="lidar_optical_joint" type="fixed">
+    <parent link="lidar_link"/>
+    <child  link="lidar_link_optical"/>
+    <origin xyz="0 0 0" rpy="0 0 0"/>
+  </joint>
   <gazebo reference="lidar_link">
-      <sensor name="gpu_lidar" type="gpu_lidar">
-        <pose relative_to="lidar_link">0 0 0 0 0 0</pose>
-        <topic>scan</topic>
-        <update_rate>10</update_rate>
-        <lidar>
-          <scan>
-            <horizontal>
-              <samples>720</samples>
-              <resolution>1</resolution>
-              <min_angle>-3.14159</min_angle>
-              <max_angle>3.14159</max_angle>
-            </horizontal>
-          </scan>
-          <range>
-            <min>0.05</min>
-            <max>12.0</max>
-            <resolution>0.005</resolution>
-          </range>
-          <noise>
-            <type>gaussian</type>
-            <mean>0.0</mean>
-            <stddev>0.001</stddev>
-          </noise>
-        </lidar>
-        <always_on>1</always_on>
-        <visualize>true</visualize>
-      </sensor>
+    <sensor name="gpu_lidar" type="gpu_lidar">
+      <pose relative_to="lidar_link">0 0 0 0 0 0</pose>
+      <topic>scan</topic>
+      <update_rate>10</update_rate>
+      <lidar>
+        <scan>
+          <horizontal>
+            <samples>720</samples>
+            <resolution>1</resolution>
+            <min_angle>-3.14159</min_angle>
+            <max_angle>3.14159</max_angle>
+          </horizontal>
+          <vertical>
+            <samples>32</samples>
+            <resolution>1</resolution>
+            <min_angle>-0.0001</min_angle>
+            <max_angle>0.0001</max_angle>
+          </vertical>
+        </scan>
+        <range>
+          <min>0.05</min>
+          <max>12.0</max>
+          <resolution>0.005</resolution>
+        </range>
+        <noise>
+          <type>gaussian</type>
+          <mean>0.0</mean>
+          <stddev>0.001</stddev>
+        </noise>
+      </lidar>
+      <always_on>1</always_on>
+      <visualize>true</visualize>
+    </sensor>
   </gazebo>
 </robot>

File: src/sweepi_description/urdf/sweepi.urdf.xacro (robot description, xacro)
@@ -5,5 +5,70 @@
   <!-- Include sensors (camera and lidar) -->
   <xacro:include filename="camera.xacro"/>
-  <xacro:include filename="lidar.xacro"/>
+  <!-- <xacro:include filename="lidar.xacro"/> -->
+  <!-- Add this to your sweepi.urdf.xacro where you currently have lidar -->
+  <!-- LIDAR Link (just geometry, no sensor) -->
+  <link name="base_scan">
+    <visual>
+      <origin xyz="0 0 0" rpy="0 0 0"/>
+      <geometry>
+        <cylinder radius="0.0508" length="0.055"/>
+      </geometry>
+      <material name="black"/>
+    </visual>
+    <collision>
+      <origin xyz="0 0 0" rpy="0 0 0"/>
+      <geometry>
+        <cylinder radius="0.0508" length="0.055"/>
+      </geometry>
+    </collision>
+    <inertial>
+      <mass value="0.114"/>
+      <origin xyz="0 0 0"/>
+      <inertia ixx="0.001" ixy="0.0" ixz="0.0" iyy="0.001" iyz="0.0" izz="0.001"/>
+    </inertial>
+  </link>
+  <!-- LIDAR Joint -->
+  <joint name="scan_joint" type="fixed">
+    <parent link="base_link"/>
+    <child link="base_scan"/>
+    <origin xyz="0.0 0.0 0.15" rpy="0 0 0"/>
+  </joint>
+  <!-- ========== GAZEBO PLUGINS ========== -->
+  <!-- LIDAR Sensor Plugin -->
+  <gazebo reference="base_scan">
+    <sensor name="scan" type="gpu_lidar">
+      <pose relative_to="base_scan">0 0 0 0 0 0</pose>
+      <topic>scan</topic>
+      <update_rate>10</update_rate>
+      <ray>
+        <scan>
+          <horizontal>
+            <samples>720</samples>
+            <resolution>1</resolution>
+            <min_angle>-3.14159</min_angle>
+            <max_angle>3.14159</max_angle>
+          </horizontal>
+          <!-- <vertical>
+            <samples>32</samples>
+            <resolution>1</resolution>
+            <min_angle>-0.5236</min_angle>
+            <max_angle>0.5236</max_angle>
+          </vertical> -->
+        </scan>
+        <range>
+          <min>0.05</min>
+          <max>12.0</max>
+          <resolution>0.005</resolution>
+        </range>
+        <noise>
+          <type>gaussian</type>
+          <mean>0.0</mean>
+          <stddev>0.001</stddev>
+        </noise>
+      </ray>
+      <always_on>1</always_on>
+      <visualize>true</visualize>
+    </sensor>
+  </gazebo>
   <!-- Include Gazebo sensor plugins -->
   <!-- <xacro:include filename="sensor_gazebo.xacro"/> -->
