Commit message: Update

File: src/sweepi_description/urdf/sweepi.urdf.xacro (robot description, xacro)
@@ -5,64 +5,30 @@
   <!-- Include sensors (camera and lidar) -->
   <xacro:include filename="camera.xacro"/>
-  <!-- <xacro:include filename="lidar.xacro"/> -->
-  <!-- Add this to your sweepi.urdf.xacro where you currently have lidar -->
-  <!-- LIDAR Link (just geometry, no sensor) -->
-  <link name="base_scan">
-    <visual>
-      <origin xyz="0 0 0" rpy="0 0 0"/>
-      <geometry>
-        <cylinder radius="0.0508" length="0.055"/>
-      </geometry>
-      <material name="black"/>
-    </visual>
-    <collision>
-      <origin xyz="0 0 0" rpy="0 0 0"/>
-      <geometry>
-        <cylinder radius="0.0508" length="0.055"/>
-      </geometry>
-    </collision>
-    <inertial>
-      <mass value="0.114"/>
-      <origin xyz="0 0 0"/>
-      <inertia ixx="0.001" ixy="0.0" ixz="0.0" iyy="0.001" iyz="0.0" izz="0.001"/>
-    </inertial>
-  </link>
-  <!-- LIDAR Joint -->
-  <joint name="scan_joint" type="fixed">
-    <parent link="base_link"/>
-    <child link="base_scan"/>
-    <origin xyz="0.0 0.0 0.15" rpy="0 0 0"/>
-  </joint>
-  <!-- ========== GAZEBO PLUGINS ========== -->
-  <!-- LIDAR Sensor Plugin -->
+  <xacro:include filename="lidar.xacro"/>
+  <!-- ========== GAZEBO LIDAR PLUGIN ========== -->
   <gazebo reference="base_scan">
     <sensor name="scan" type="gpu_lidar">
       <pose relative_to="base_scan">0 0 0 0 0 0</pose>
       <topic>scan</topic>
-      <update_rate>10</update_rate>
+      <frame_name>base_scan</frame_name>
+      <update_rate>5.5</update_rate>
       <ray>
         <scan>
           <horizontal>
-            <samples>720</samples>
+            <samples>1200</samples>
             <resolution>1</resolution>
-            <min_angle>-3.14159</min_angle>
-            <max_angle>3.14159</max_angle>
+            <min_angle>-3.14159265</min_angle>
+            <max_angle>3.14159265</max_angle>
           </horizontal>
-          <!-- <vertical>
-            <samples>32</samples>
-            <resolution>1</resolution>
-            <min_angle>-0.5236</min_angle>
-            <max_angle>0.5236</max_angle>
-          </vertical> -->
         </scan>
         <range>
-          <min>0.05</min>
-          <max>12.0</max>
-          <resolution>0.005</resolution>
+          <min>0.15</min>
+          <max>8.0</max>
+          <resolution>0.01</resolution>
         </range>
         <noise>
           <type>gaussian</type>
           <mean>0.0</mean>
-          <stddev>0.001</stddev>
+          <stddev>0.01</stddev>
         </noise>
       </ray>
@@ -71,6 +37,4 @@
     </sensor>
   </gazebo>
-  <!-- Include Gazebo sensor plugins -->
-  <!-- <xacro:include filename="sensor_gazebo.xacro"/> -->
   <!-- Include Gazebo base plugins and controller -->
   <xacro:include filename="robot_base_gazebo.xacro"/>
