Commit message: Update: fixed real robot issues ( disabled imu readings)

File: src/sweepi_description/urdf/robot_base.xacro (robot description, xacro)
@@ -4,7 +4,7 @@
   <xacro:property name="body_height"        value="0.100" />
   <xacro:property name="ground_clearance"   value="0.020" />
-  <xacro:property name="drive_wheel_radius" value="0.025" />
+  <xacro:property name="drive_wheel_radius" value="0.0615" />
   <xacro:property name="drive_wheel_width"  value="0.020" />
-  <xacro:property name="wheel_span"         value="0.300" />
+  <xacro:property name="wheel_span"         value="0.290" />
   <xacro:property name="caster_offset_x"    value="0.160" />
   <xacro:property name="caster_radius"      value="${ground_clearance / 2.0}" />

File: src/sweepi_description/urdf/robot_base_gazebo.xacro (robot description, xacro)
@@ -16,6 +16,6 @@
       <left_joint>base_left_wheel_joint</left_joint>
       <right_joint>base_right_wheel_joint</right_joint>
-      <wheel_separation>0.300</wheel_separation>
-      <wheel_radius>0.025</wheel_radius>
+      <wheel_separation>0.290</wheel_separation>
+      <wheel_radius>0.0615</wheel_radius>
       <odom_publish_frequency>50</odom_publish_frequency>
       <topic>/model/sweepi/cmd_vel</topic>
